File: mm_motor.kicad_sch (KiCad schematic)
At the start: 1 part, among them M1 N20_encoder

Commit message: tp2
Parts:
- added J3: Conn_01x06, Connector_PinHeader_2.54mm:PinHeader_1x06_P2.54mm_Vertical, symbol Connector_Generic:Conn_01x06
Connections:
- net C1: now also J3.3 (Pin_3)
- net C2: now also J3.4 (Pin_4)
- net MA: now also J3.1 (Pin_1)
- net MB: now also J3.6 (Pin_6)
- new net +BATT: J3.5 (Pin_5)
- new net GND: J3.2 (Pin_2)
Other:
- moved on the sheet: M1
Changed lines of the file:
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@@
 (kicad_sch (version 20230121) (generator eeschema)
   (paper "A4")
-  (hierarchical_label "C1" (shape output) (at 118.11 91.44 180) (fields_autoplaced)
+  (wire (pts (xy 157.48 82.55) (xy 167.64 82.55))
+    (stroke (width 0) (type default))
+  )
+  (wire (pts (xy 157.48 80.01) (xy 167.64 80.01))
+    (stroke (width 0) (type default))
+  )
+  (wire (pts (xy 142.24 77.47) (xy 142.24 82.55))
+    (stroke (width 0) (type default))
+  )
+  (wire (pts (xy 167.64 77.47) (xy 142.24 77.47))
+    (stroke (width 0) (type default))
+  )
+  (wire (pts (xy 167.64 85.09) (xy 148.59 85.09))
+    (stroke (width 0) (type default))
+  )
+  (wire (pts (xy 157.48 87.63) (xy 167.64 87.63))
+    (stroke (width 0) (type default))
+  )
+  (wire (pts (xy 157.48 74.93) (xy 167.64 74.93))
+    (stroke (width 0) (type default))
+  )
+  (wire (pts (xy 148.59 85.09) (xy 148.59 83.82))
+    (stroke (width 0) (type default))
+  )
+  (hierarchical_label "C1" (shape output) (at 157.48 80.01 180) (fields_autoplaced)
     (effects (font (size 1.27 1.27)) (justify right))
   )
-  (hierarchical_label "C2" (shape output) (at 118.11 93.98 180) (fields_autoplaced)
+  (hierarchical_label "C2" (shape output) (at 157.48 82.55 180) (fields_autoplaced)
     (effects (font (size 1.27 1.27)) (justify right))
   )
-  (hierarchical_label "MB" (shape passive) (at 118.11 99.06 180) (fields_autoplaced)
+  (hierarchical_label "MB" (shape passive) (at 157.48 87.63 180) (fields_autoplaced)
     (effects (font (size 1.27 1.27)) (justify right))
   )
-  (hierarchical_label "MA" (shape passive) (at 118.11 86.36 180) (fields_autoplaced)
+  (hierarchical_label "MA" (shape passive) (at 157.48 74.93 180) (fields_autoplaced)
     (effects (font (size 1.27 1.27)) (justify right))
   )
-  (symbol (lib_id "minimouse:N20_w_encoder") (at 115.57 57.15 0) (unit 1)
+  (symbol (lib_id "power:+BATT") (at 148.59 83.82 0) (unit 1)
     (in_bom yes) (on_board yes) (dnp no) (fields_autoplaced)
-    (property "Reference" "M1" (at 118.11 55.88 0)
+    (property "Reference" "#PWR031" (at 148.59 87.63 0)
+      (effects (font (size 1.27 1.27)) hide)
+    )
+    (property "Value" "+BATT" (at 148.59 78.74 0)
+      (effects (font (size 1.27 1.27)))
+    )
+    (property "Footprint" "" (at 148.59 83.82 0)
+      (effects (font (size 1.27 1.27)) hide)
+    )
+    (property "Datasheet" "" (at 148.59 83.82 0)
+      (effects (font (size 1.27 1.27)) hide)
+    )
+    (pin "1")
+    (instances
+      (project "minimouse"
+        (path "/d8fa4cba-2469-4231-847f-065b6b829f44/7f113667-692a-4f4d-b16f-621d32f3f136"
+          (reference "#PWR031") (unit 1)
+        )
+        (path "/d8fa4cba-2469-4231-847f-065b6b829f44/3975acd0-18ad-47bc-9ce1-d8c4d864aafe"
+          (reference "#PWR032") (unit 1)
+        )
+      )
+    )
+  )
+  (symbol (lib_id "power:GND") (at 142.24 82.55 0) (unit 1)
+    (in_bom yes) (on_board yes) (dnp no) (fields_autoplaced)
+    (property "Reference" "#PWR029" (at 142.24 88.9 0)
+      (effects (font (size 1.27 1.27)) hide)
+    )
+    (property "Value" "GND" (at 142.24 87.63 0)
+      (effects (font (size 1.27 1.27)))
+    )
+    (property "Footprint" "" (at 142.24 82.55 0)
+      (effects (font (size 1.27 1.27)) hide)
+    )
+    (property "Datasheet" "" (at 142.24 82.55 0)
+      (effects (font (size 1.27 1.27)) hide)
+    )
+    (pin "1")
+    (instances
+      (project "minimouse"
+        (path "/d8fa4cba-2469-4231-847f-065b6b829f44/7f113667-692a-4f4d-b16f-621d32f3f136"
+          (reference "#PWR029") (unit 1)
+        )
+        (path "/d8fa4cba-2469-4231-847f-065b6b829f44/3975acd0-18ad-47bc-9ce1-d8c4d864aafe"
+          (reference "#PWR030") (unit 1)
+        )
+      )
+    )
+  )
+  (symbol (lib_id "minimouse:N20_w_encoder") (at 154.94 45.72 0) (unit 1)
+    (in_bom yes) (on_board yes) (dnp no) (fields_autoplaced)
+    (property "Reference" "M1" (at 157.48 44.45 0)
       (effects (font (size 1.27 1.27)) (justify left))
     )
-    (property "Value" "N20_encoder" (at 118.11 58.42 0)
+    (property "Value" "N20_encoder" (at 157.48 46.99 0)
       (effects (font (size 1.27 1.27)) (justify left))
     )
-    (property "Footprint" "minimouse:N20_with_encoder" (at 118.11 53.34 0)
+    (property "Footprint" "minimouse:N20_with_encoder" (at 157.48 41.91 0)
       (effects (font (size 1.27 1.27)) hide)
     )
-    (property "Datasheet" "" (at 115.57 57.15 0)
+    (property "Datasheet" "" (at 154.94 45.72 0)
       (effects (font (size 1.27 1.27)) hide)
     )
@@
         )
       )
+    )
+  )
+  (symbol (lib_id "Connector_Generic:Conn_01x06") (at 172.72 80.01 0) (unit 1)
+    (in_bom yes) (on_board yes) (dnp no) (fields_autoplaced)
+    (property "Reference" "J3" (at 175.26 80.01 0)
+      (effects (font (size 1.27 1.27)) (justify left))
+    )
+    (property "Value" "Conn_01x06" (at 175.26 82.55 0)
+      (effects (font (size 1.27 1.27)) (justify left))
+    )
+    (property "Footprint" "Connector_PinHeader_2.54mm:PinHeader_1x06_P2.54mm_Vertical" (at 172.72 80.01 0)
+      (effects (font (size 1.27 1.27)) hide)
+    )
+    (property "Datasheet" "~" (at 172.72 80.01 0)
+      (effects (font (size 1.27 1.27)) hide)
+    )
+    (pin "1")
+    (pin "5")
+    (pin "4")
+    (pin "3")
+    (pin "6")
+    (pin "2")
+    (instances
+      (project "minimouse"
+        (path "/d8fa4cba-2469-4231-847f-065b6b829f44/7f113667-692a-4f4d-b16f-621d32f3f136"
+          (reference "J3") (unit 1)
+        )
+        (path "/d8fa4cba-2469-4231-847f-065b6b829f44/3975acd0-18ad-47bc-9ce1-d8c4d864aafe"
+          (reference "J4") (unit 1)
+        )
+      )
