File: mm_motor_control.kicad_sch (KiCad schematic)
At the start: 0 parts

Commit message: tp2
Parts:
- added C10: 2.2µF, symbol Device:C
- added C11: 22µF, symbol Device:C
- added C7: C, symbol Device:C
- added C8: 22nF, symbol Device:C
- added C9: 10nF, symbol Device:C
- added R10, R15: 18K, Resistor_SMD:R_0603_1608Metric, symbol Device:R
- added R11, R12: 10K, Resistor_SMD:R_0603_1608Metric, symbol Device:R
- added R13: 1K, Resistor_SMD:R_0603_1608Metric, symbol Device:R
- added R14: 47K, Resistor_SMD:R_0603_1608Metric, symbol Device:R
- added R16, R17: 330m, Resistor_SMD:R_0603_1608Metric, symbol Device:R
- added U2: STSPIN240, Package_DFN_QFN:VQFN-16-1EP_3x3mm_P0.5mm_EP1.8x1.8mm, symbol Driver_Motor:STSPIN240
Connections:
- net EN: now also R15.2
- net FAULT: now also C9.1, R15.1, U2.13 (EN/FLT)
- net OUT_A1: now also U2.3 (OUTA1)
- net OUT_A2: now also U2.5 (OUTA2)
- net OUT_B1: now also U2.10 (OUTB1)
- net OUT_B2: now also U2.8 (OUTB2)
- net PHASE_A: now also U2.1 (PHA)
- net PHASE_B: now also U2.15 (PHB)
- net PWM_A: now also U2.2 (PWMA)
- net PWM_B: now also U2.16 (PWMB)
- net STBY/RESET: now also C7.1, R10.2, U2.14 (STBY/RESET)
- new net: C8.1, R13.2
- new net: R11.2, R12.1, U2.11 (REF)
- new net: R13.1, R14.1, U2.12 (TOFF)
- new net: R16.1, U2.4 (SENSEA)
- new net: R17.1, U2.9 (SENSEB)
- new net +3.3V: R10.1
- new net +BATT: R11.1
- new net GND: C10.2, C11.2, C7.2, C8.2, C9.2, R12.2, R14.2, R16.2, R17.2
- new net VS: C10.1, C11.1, U2.6 (VS)
